Commit message: too strong

File: SpiderBot/spider.urdf (robot description, URDF)
Before this commit: robot blocky_spider, 31 links, 30 joints
Links:
- link leg_foot_0: mass 0.000000 -> 0.011570
- link leg_foot_1: mass 0.000000 -> 0.011570
- link leg_foot_2: mass 0.000000 -> 0.011570
- link leg_foot_3: mass 0.000000 -> 0.011570
- link leg_foot_4: mass 0.000000 -> 0.011570
- link leg_foot_5: mass 0.000000 -> 0.011570
